Commit message: update

File: ros2/xiaoxdummy_ws/src/xiaoxdummy_control/config/xiaoxdummy.urdf (robot description, URDF)
Before this commit: robot xiaoxdummy, 7 links, 6 joints
Links:
- link Base_Link: geometry collision mesh filename=file:///home/jiehuang/xiaoxdummy/ros2/xiaoxdummy_ws/src/xia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; visual mesh filename=file:///home/jiehuang/xiaoxdummy/ros2/xiaoxdummy_ws/src/xia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
- link Link1: geometry collision mesh filename=file:///home/jiehuang/xiaoxdummy/ros2/xiaoxdummy_ws/src/xia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; visual mesh filename=file:///home/jiehuang/xiaoxdummy/ros2/xiaoxdummy_ws/src/xia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
- link Link2: geometry collision mesh filename=file:///home/jiehuang/xiaoxdummy/ros2/xiaoxdummy_ws/src/xia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; visual mesh filename=file:///home/jiehuang/xiaoxdummy/ros2/xiaoxdummy_ws/src/xia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
- link Link3: geometry collision mesh filename=file:///home/jiehuang/xiaoxdummy/ros2/xiaoxdummy_ws/src/xia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; visual mesh filename=file:///home/jiehuang/xiaoxdummy/ros2/xiaoxdummy_ws/src/xia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
- link Link4: geometry collision mesh filename=file:///home/jiehuang/xiaoxdummy/ros2/xiaoxdummy_ws/src/xia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; visual mesh filename=file:///home/jiehuang/xiaoxdummy/ros2/xiaoxdummy_ws/src/xia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
- link Link5: geometry collision mesh filename=file:///home/jiehuang/xiaoxdummy/ros2/xiaoxdummy_ws/src/xia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; visual mesh filename=file:///home/jiehuang/xiaoxdummy/ros2/xiaoxdummy_ws/src/xia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
- link Link6: geometry collision mesh filename=file:///home/jiehuang/xiaoxdummy/ros2/xiaoxdummy_ws/src/xia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; visual mesh filename=file:///home/jiehuang/xiaoxdummy/ros2/xiaoxdummy_ws/src/xia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

Commit message: update

File: ros2/xiaoxdummy_ws/src/xiaoxdummy_control/config/xiaoxdummy.urdf (robot description, URDF)
Before this commit: robot xiaoxdummy, 7 links, 6 joints
Links:
- link Base_Link: geometry collision mesh filename=package://xiaoxdummy_control/meshes/base_link.stl; visual mesh filename=package://xiaoxdummy_control/meshes/base_link.stl
- link Link1: geometry collision mesh filename=package://xiaoxdummy_control/meshes/link1.stl; visual mesh filename=package://xiaoxdummy_control/meshes/link1.stl
- link Link2: geometry collision mesh filename=package://xiaoxdummy_control/meshes/link2.stl; visual mesh filename=package://xiaoxdummy_control/meshes/link2.stl
- link Link3: geometry collision mesh filename=package://xiaoxdummy_control/meshes/link3.stl; visual mesh filename=package://xiaoxdummy_control/meshes/link3.stl
- link Link4: geometry collision mesh filename=package://xiaoxdummy_control/meshes/link4.stl; visual mesh filename=package://xiaoxdummy_control/meshes/link4.stl
- link Link5: geometry collision mesh filename=package://xiaoxdummy_control/meshes/link5.stl; visual mesh filename=package://xiaoxdummy_control/meshes/link5.stl
- link Link6: geometry collision mesh filename=package://xiaoxdummy_control/meshes/link6.stl; visual mesh filename=package://xiaoxdummy_control/meshes/link6.stl

File: ros2/xiaoxdummy_ws/src/xiaoxdummy_control/config/xiaoxdummy_ros2_control.xacro (robot description, xacro)
@@ -49,15 +49,12 @@
   <ros2_control name="XiaoxdummySystem" type="system">
     <hardware>
-      <xacro:if value="$(arg use_real_hardware)">
-        <plugin>xiaoxdummy_control/XiaoxdummyHardwareInterface</plugin>
-        <param name="serial_port">$(arg serial_port)</param>
-        <param name="baud_rate">$(arg baud_rate)</param>
-        <param name="command_speed">$(arg command_speed)</param>
+      <xacro:if value="$(arg use_gazebo)">
+        <plugin>gz_ros2_control/GazeboSimSystem</plugin>
       </xacro:if>
-      <xacro:unless value="$(arg use_real_hardware)">
-        <xacro:if value="$(arg use_gazebo)">
-          <plugin>gz_ros2_control/GazeboSimSystem</plugin>
+      <xacro:unless value="$(arg use_gazebo)">
+        <xacro:if value="$(arg use_real_hardware)">
+          <plugin>xiaoxdummy_hw/XiaoxdummyHardware</plugin>
         </xacro:if>
-        <xacro:unless value="$(arg use_gazebo)">
+        <xacro:unless value="$(arg use_real_hardware)">
           <plugin>mock_components/GenericSystem</plugin>
         </xacro:unless>

Commit message: 添加limit和direction

File: ros2/xiaoxdummy_ws/src/xiaoxdummy_control/config/xiaoxdummy.urdf (robot description, URDF)
Before this commit: robot xiaoxdummy, 7 links, 6 joints
Joints:
- joint Joint1: limit (none) -> lower=-3.001966 upper=3.001966 effort=100 velocity=100; type continuous -> revolute
- joint Joint2: limit (none) -> lower=-1.570796 upper=1.308997 effort=100 velocity=100; type continuous -> revolute
- joint Joint3: limit (none) -> lower=-1.500983 upper=1.570796 effort=100 velocity=100; type continuous -> revolute
- joint Joint4: limit (none) -> lower=-3.141593 upper=3.141593 effort=100 velocity=100; type continuous -> revolute
- joint Joint5: limit (none) -> lower=-1.919862 upper=2.094395 effort=100 velocity=100; type continuous -> revolute
- joint Joint6: limit (none) -> lower=-3.141593 upper=3.141593 effort=100 velocity=100; type continuous -> revolute

File: ros2/xiaoxdummy_ws/src/xiaoxdummy_control/config/xiaoxdummy_ros2_control.xacro (robot description, xacro)
@@ -73,5 +73,5 @@
     <!-- Joint2 -->
     <joint name="Joint2">
-      <param name="direction">-1.0</param>
+      <param name="direction">1.0</param>
       <command_interface name="position"/>
       <state_interface name="position">
